File: file5BCDBE1F.sch (KiCad schematic (older format))
At the start: 31 parts, among them J3 Jack-DC, Q3 Q_NMOS_GDS, SW1 SW_DPST_x2, U5 ATTINY85-20SU, U6 PCF8523, U7 TPS630701, Y2 32.768

Commit message: deleted unused files and tidied up footprint librarys
Parts:
- SW1: footprint switch-footprint:CJS-1200A1 -> pi-hat-footprints:CJS-1200A1
Changed lines of the file:
@@
 F 0 "SW1" H 2550 6185 50  0000 C CNN
 F 1 "SW_DPST_x2" H 2550 6094 50  0000 C CNN
-F 2 "switch-footprint:CJS-1200A1" H 2550 5950 50  0001 C CNN
+F 2 "pi-hat-footprints:CJS-1200A1" H 2550 5950 50  0001 C CNN
 F 3 "" H 2550 5950 50  0001 C CNN
 F 4 "563-1021-1-ND" H 2550 5950 50  0001 C CNN "Digikey"

Commit message: Added link, MPN, and Digikey number to all parts.
Parts:
- BT2: Digikey BC501SM-ND, SY033-ND -> BC501SM-ND; Digikey2 SY033-ND -> (none); Link (none) -> https://www.digikey.com/product-detail/en/mpd-memory-protec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; MPN (none) -> BC501SM
- C1, C2: Digikey (none) -> 1276-1066-1-ND; Link (none) -> https://www.digikey.com/product-detail/en/samsung-electro-m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; MPN (none) -> CL21B105KAFNNNE
- C11: symbol pi-hat-rescue:CP-Device -> pi-hat-rescue:CP-Device-pi-hat-rescue; Link (none) -> https://www.digikey.com/product-detail/en/rubycon/25ZLH820M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; MPN (none) -> 25ZLH820MEFC10X20
- C12, C19, C20: Digikey (none) -> 1276-2891-1-ND; Link (none) -> https://www.digikey.com/product-detail/en/samsung-electro-m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; MPN (none) -> CL21A106KAYNNNE
- C13, C14, C15: Digikey (none) -> 490-12389-1-ND; Link (none) -> https://www.digikey.com/product-detail/en/murata-electronic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; MPN (none) -> GRT21BR61E226ME13L
- C16: Digikey (none) -> 720-1756-1-ND; Link (none) -> https://www.digikey.com/product-detail/en/vishay-vitramon/V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; MPN (none) -> VJ0805Y104MXXAT
- C17, C18: Digikey (none) -> 445-11238-1-ND; Link (none) -> https://www.digikey.com/product-detail/en/tdk-corporation/C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; MPN (none) -> C1608JB1E106M080AC
- D2: symbol pi-hat-rescue:LED-Device -> pi-hat-rescue:LED-Device-pi-hat-rescue; Link (none) -> https://www.digikey.com/product-detail/en/lite-on-inc/LTST-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; MPN (none) -> LTST-C191KGKT
- D3: Link (none) -> https://www.digikey.com/product-detail/en/on-semiconductor/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; MPN (none) -> MM3Z4V3B
- D4: Link (none) -> https://www.digikey.com/product-detail/en/micro-commercial-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; MPN (none) -> 1N4148WX-TP
- J3: symbol pi-hat-rescue:Connector_Specialized_Jack-DC-pi-hat-cache -> pi-hat-rescue:Connector_Specialized_Jack-DC-pi-hat-cache-pi-hat-rescue; Link (none) -> https://www.digikey.com/product-detail/en/cui-inc/PJ-002A/C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; MPN (none) -> PJ-002A
- L2: Link (none) -> https://www.digikey.com/product-detail/en/panasonic-electro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; MPN (none) -> ETQ-P3M1R5KVP
- Q3: symbol pi-hat-rescue:Q_NMOS_GDSD-Device -> pi-hat-rescue:Q_NMOS_GDSD-Device-pi-hat-rescue; Link (none) -> https://www.digikey.com/product-detail/en/on-semiconductor/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; MPN (none) -> NTF3055L108T1G
- R1, R16: Digikey 311-1.0KGRCT-ND -> P1.00KHCT-ND; Link (none) -> https://www.digikey.com/product-detail/en/panasonic-electro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; MPN (none) -> ERJ-3EKF1001V
- R17: Digikey (none) -> RR08P100KDCT-ND; Link (none) -> https://www.digikey.com/product-detail/en/susumu/RR0816P-10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; MPN (none) -> RR0816P-104-D
- R18, R4: Digikey (none) -> A126394CT-ND; Link (none) -> https://www.digikey.com/product-detail/en/te-connectivity-p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; MPN (none) -> CRGH0603J10K
- R6: symbol pi-hat-rescue:R-Device -> pi-hat-rescue:R-Device-pi-hat-rescue; Digikey (none) -> 311-470HRCT-ND; Link (none) -> https://www.digikey.com/product-detail/en/yageo/RC0603FR-07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; MPN (none) -> RC0603FR-07470RL
- R9: symbol pi-hat-rescue:R-Device -> pi-hat-rescue:R-Device-pi-hat-rescue; Digikey (none) -> RR08P100KDCT-ND; Link (none) -> https://www.digikey.com/product-detail/en/susumu/RR0816P-10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; MPN (none) -> RR0816P-104-D
- SW1: Link (none) -> https://www.digikey.com/product-detail/en/nidec-copal-elect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; MPN (none) -> CJS-1200TA
- U5: symbol pi-hat-rescue:ATTINY85-20SU-pi-hat-cache -> pi-hat-rescue:ATTINY85-20SU-pi-hat-cache-pi-hat-rescue; Link (none) -> https://www.digikey.com/product-detail/en/assmann-wsw-compo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; MPN (none) -> A 08-LC-TT
- U6: Link (none) -> https://www.digikey.com/product-detail/en/nxp-usa-inc/PCF85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; MPN (none) -> PCF8523T/1,118
- U7: Digikey (none) -> 296-44765-1-ND; Link (none) -> https://www.digikey.com/product-detail/en/texas-instruments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; MPN (none) -> TPS630701RNMT
- Y2: Link (none) -> https://www.digikey.com/product-detail/en/abracon-llc/ABS25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; MPN (none) -> ABS25-32.768KHZ-6-T

Commit message: Added some Seeed OPL parts
Parts:
- C1, C2: OPL (none) -> CC0805KKX7R8BB105
- C12, C19, C20: OPL (none) -> CC0805KKX5R8BB106
- C13, C14, C15: OPL (none) -> CL21A226MQQNNNE
- C16: OPL (none) -> CC0805KRX7R9BB104
- C17, C18: OPL (none) -> CC0603KRX5R6BB106
- J3: OPL (none) -> DC-005
- R1, R16: OPL (none) -> RC0603JR-071KL
- R17, R9: OPL (none) -> RC0603JR-07100KL
- R18, R4: OPL (none) -> SMD RES 10K-5%-1/10W
- R6: OPL (none) -> RC0603JR-07470RL
Changed lines of the file:
@@
 F 5 "https://www.digikey.com/product-detail/en/cui-inc/PJ-002A/CP-002A-ND/96962" H 0   0   50  0001 C CNN "Link"
 F 6 "PJ-002A" H 0   0   50  0001 C CNN "MPN"
+F 7 "DC-005" H 0   0   50  0001 C CNN "OPL"
 	1    1050 2550
 	1    0    0    -1
@@
 F 5 "https://www.digikey.com/product-detail/en/susumu/RR0816P-104-D/RR08P100KDCT-ND/432772" H 0   0   50  0001 C CNN "Link"
 F 6 "RR0816P-104-D" H 0   0   50  0001 C CNN "MPN"
+F 7 "RC0603JR-07100KL" H 0   0   50  0001 C CNN "OPL"
 	1    3000 6150
 	1    0    0    -1
@@
 F 5 "https://www.digikey.com/product-detail/en/yageo/RC0603FR-07470RL/311-470HRCT-ND/730203" H 0   0   50  0001 C CNN "Link"
 F 6 "RC0603FR-07470RL" H 0   0   50  0001 C CNN "MPN"
+F 7 "RC0603JR-07470RL" H 0   0   50  0001 C CNN "OPL"
 	1    2700 4700
 	0    1    1    0
@@
 F 5 "https://www.digikey.com/product-detail/en/te-connectivity-passive-product/CRGH0603J10K/A126394CT-ND/7603449" H 0   0   50  0001 C CNN "Link"
 F 6 "CRGH0603J10K" H 0   0   50  0001 C CNN "MPN"
+F 7 "SMD RES 10K-5%-1/10W" H 0   0   50  0001 C CNN "OPL"
 	1    9900 4950
 	0    1    1    0
@@
 F 5 "https://www.digikey.com/product-detail/en/samsung-electro-mechanics/CL21A106KAYNNNE/1276-2891-1-ND/3890977" H 0   0   50  0001 C CNN "Link"
 F 6 "CL21A106KAYNNNE" H 0   0   50  0001 C CNN "MPN"
+F 7 "CC0805KKX5R8BB106" H 0   0   50  0001 C CNN "OPL"
 	1    10800 5200
 	1    0    0    -1
@@
 F 5 "https://www.digikey.com/product-detail/en/samsung-electro-mechanics/CL21A106KAYNNNE/1276-2891-1-ND/3890977" H 0   0   50  0001 C CNN "Link"
 F 6 "CL21A106KAYNNNE" H 0   0   50  0001 C CNN "MPN"
+F 7 "CC0805KKX5R8BB106" H 0   0   50  0001 C CNN "OPL"
 	1    10450 5200
 	1    0    0    -1
@@
 F 5 "https://www.digikey.com/product-detail/en/tdk-corporation/C1608JB1E106M080AC/445-11238-1-ND/3952904" H 0   0   50  0001 C CNN "Link"
 F 6 "C1608JB1E106M080AC" H 0   0   50  0001 C CNN "MPN"
+F 7 "CC0603KRX5R6BB106" H 0   0   50  0001 C CNN "OPL"
 	1    10050 5200
 	1    0    0    -1
@@
 F 5 "https://www.digikey.com/product-detail/en/vishay-vitramon/VJ0805Y104MXXAT/720-1756-1-ND/8324176" H 0   0   50  0001 C CNN "Link"
 F 6 "VJ0805Y104MXXAT" H 0   0   50  0001 C CNN "MPN"
+F 7 "CC0805KRX7R9BB104" H 0   0   50  0001 C CNN "OPL"
 	1    8200 4950
 	0    1    1    0
@@
 F 5 "https://www.digikey.com/product-detail/en/susumu/RR0816P-104-D/RR08P100KDCT-ND/432772" H 0   0   50  0001 C CNN "Link"
 F 6 "RR0816P-104-D" H 0   0   50  0001 C CNN "MPN"
+F 7 "RC0603JR-07100KL" V 7750 5100 50  0001 C CNN "OPL"
 	1    7750 5100
 	-1   0    0    1
@@
 F 5 "https://www.digikey.com/product-detail/en/murata-electronics-north-america/GRT21BR61E226ME13L/490-12389-1-ND/5417090" H 0   0   50  0001 C CNN "Link"
 F 6 "GRT21BR61E226ME13L" H 0   0   50  0001 C CNN "MPN"
+F 7 "CL21A226MQQNNNE" H 0   0   50  0001 C CNN "OPL"
 	1    7300 5650
 	1    0    0    -1
@@
 F 5 "https://www.digikey.com/product-detail/en/murata-electronics-north-america/GRT21BR61E226ME13L/490-12389-1-ND/5417090" H 0   0   50  0001 C CNN "Link"
 F 6 "GRT21BR61E226ME13L" H 0   0   50  0001 C CNN "MPN"
+F 7 "CL21A226MQQNNNE" H 0   0   50  0001 C CNN "OPL"
 	1    7650 5650
 	1    0    0    -1
@@
 F 5 "https://www.digikey.com/product-detail/en/murata-electronics-north-america/GRT21BR61E226ME13L/490-12389-1-ND/5417090" H 0   0   50  0001 C CNN "Link"
 F 6 "GRT21BR61E226ME13L" H 0   0   50  0001 C CNN "MPN"
+F 7 "CL21A226MQQNNNE" H 0   0   50  0001 C CNN "OPL"
 	1    8100 5650
 	1    0    0    -1
@@
 F 5 "https://www.digikey.com/product-detail/en/tdk-corporation/C1608JB1E106M080AC/445-11238-1-ND/3952904" H 0   0   50  0001 C CNN "Link"
 F 6 "C1608JB1E106M080AC" H 0   0   50  0001 C CNN "MPN"
+F 7 "CC0603KRX5R6BB106" H 0   0   50  0001 C CNN "OPL"
 	1    8450 5650
 	1    0    0    -1
@@
 F 5 "https://www.digikey.com/product-detail/en/panasonic-electronic-components/ERJ-3EKF1001V/P1.00KHCT-ND/198071" H 0   0   50  0001 C CNN "Link"
 F 6 "ERJ-3EKF1001V" H 0   0   50  0001 C CNN "MPN"
+F 7 "RC0603JR-071KL" H 0   0   50  0001 C CNN "OPL"
 	1    10250 1600
 	1    0    0    -1
@@
 F 5 "https://www.digikey.com/product-detail/en/samsung-electro-mechanics/CL21A106KAYNNNE/1276-2891-1-ND/3890977" H 0   0   50  0001 C CNN "Link"
 F 6 "CL21A106KAYNNNE" H 0   0   50  0001 C CNN "MPN"
+F 7 "CC0805KKX5R8BB106" H 0   0   50  0001 C CNN "OPL"
 	1    10250 2000
 	1    0    0    -1
@@
 F 5 "https://www.digikey.com/product-detail/en/panasonic-electronic-components/ERJ-3EKF1001V/P1.00KHCT-ND/198071" H 0   0   50  0001 C CNN "Link"
 F 6 "ERJ-3EKF1001V" H 0   0   50  0001 C CNN "MPN"
+F 7 "RC0603JR-071KL" H 0   0   50  0001 C CNN "OPL"
 	1    1100 5600
 	1    0    0    -1
@@
 F 5 "https://www.digikey.com/product-detail/en/te-connectivity-passive-product/CRGH0603J10K/A126394CT-ND/7603449" H 0   0   50  0001 C CNN "Link"
 F 6 "CRGH0603J10K" H 0   0   50  0001 C CNN "MPN"
+F 7 "SMD RES 10K-5%-1/10W" H 0   0   50  0001 C CNN "OPL"
 	1    1100 6000
 	1    0    0    -1
@@
 F 5 "https://www.digikey.com/product-detail/en/samsung-electro-mechanics/CL21B105KAFNNNE/1276-1066-1-ND/3889152" H 0   0   50  0001 C CNN "Link"
 F 6 "CL21B105KAFNNNE" H 0   0   50  0001 C CNN "MPN"
+F 7 "CC0805KKX7R8BB105" H 0   0   50  0001 C CNN "OPL"
 	1    1350 6000
 	1    0    0    -1
@@
 F 5 "https://www.digikey.com/product-detail/en/samsung-electro-mechanics/CL21B105KAFNNNE/1276-1066-1-ND/3889152" H 0   0   50  0001 C CNN "Link"
 F 6 "CL21B105KAFNNNE" H 0   0   50  0001 C CNN "MPN"
+F 7 "CC0805KKX7R8BB105" H 0   0   50  0001 C CNN "OPL"
 	1    6250 4850
 	1    0    0    -1

Commit message: Updated to version 0.3
Parts:
- removed BT2: 1206, pi-hat-footprints:CR1220, symbol device:Battery_Cell
- removed C1, C2: 1uF, Capacitors_SMD:C_0805_HandSoldering, symbol device:C_Small
- removed C12: 10uF, Capacitors_SMD:C_0805_HandSoldering, symbol device:C_Small
- removed D2: LED_GREEN, LEDs:LED_0603_HandSoldering, symbol pi-hat-rescue:LED-Device-pi-hat-rescue
- removed D3: D_Zener, Diodes_SMD:D_SOD-323_HandSoldering, symbol device:D_Zener
- removed D4: D, Diodes_SMD:D_SOD-323_HandSoldering, symbol device:D
- removed Q3: Q_NMOS_GDS, TO_SOT_Packages_SMD:SOT-223, symbol pi-hat-rescue:Q_NMOS_GDSD-Device-pi-hat-rescue
- removed R1, R16: 1K, Resistors_SMD:R_0603_HandSoldering, symbol device:R
- removed R4: 10K, Resistors_SMD:R_0603_HandSoldering, symbol device:R
- removed R6: 470R, Resistors_SMD:R_0603_HandSoldering, symbol pi-hat-rescue:R-Device-pi-hat-rescue
- removed R9: 100K, Resistors_SMD:R_0603_HandSoldering, symbol pi-hat-rescue:R-Device-pi-hat-rescue
- removed SW1: SW_DPST_x2, pi-hat-footprints:CJS-1200A1, symbol switches:SW_DPST_x2
- removed U5: ATTINY85-20SU, Housings_DIP:DIP-8_W7.62mm_Socket, symbol pi-hat-rescue:ATTINY85-20SU-pi-hat-cache-pi-hat-rescue
- removed U6: PCF8523, Housings_SOIC:SOIC-8_3.9x4.9mm_Pitch1.27mm, symbol cacophony-pi-hat:PCF8523
- removed Y2: 32.768, Crystals:Crystal_SMD_SeikoEpson_MC306-4pin_8.0x3.2mm_HandSoldering, symbol device:Crystal_GND23
- added C7, C8: 2.2uF, Capacitors_SMD:C_0603, symbol Device:C_Small
- added F1: Fuse, Resistors_SMD:R_0603_HandSoldering, symbol Device:Fuse
- added Q3: Q_PMOS_DGS, digikey-footprints:IRF9310PbF, symbol Device:Q_PMOS_DGS
- added R10: 100K, Resistors_SMD:R_0603, symbol Device:R
- added U3: AP2210N-3.3TRG1, TO_SOT_Packages_SMD:SOT-23, symbol cacophony-pi-hat:AP2210N-3.3TRG1
- C13, C14, C15, C16, C19, C20: footprint Capacitors_SMD:C_0805_HandSoldering -> Capacitors_SMD:C_0805
- C17, C18: footprint Capacitors_SMD:C_0603_HandSoldering -> Capacitors_SMD:C_0603; Digikey 445-11238-1-ND -> 490-7202-1-ND; Link https://www.digikey.com/product-detail/en/tdk-corporation/C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 -> https://www.digikey.com/product-detail/en/murata-electronic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; MPN C1608JB1E106M080AC -> GRM188R61E106MA73D
- R17: footprint Resistors_SMD:R_0603_HandSoldering -> Resistors_SMD:R_0603; OPL RC0603JR-07100KL -> (none)
- R18: footprint Resistors_SMD:R_0603_HandSoldering -> Resistors_SMD:R_0603
Connections:
- net Ground is gone; now on net GND: C11.2, C13.2, C14.2, C15.2, C16.2, C17.2, C18.2, C19.2, C20.2, J3.2, J3.3, U7.10 (PGND), U7.15 (VSEL), U7.4 (GND), U7.6 (FB2)
- net GND: now also C7.2, C8.2, Q3.2 (G), R10.2, U3.1 (GND)
- net VCC: now also C7.1, Q3.3 (S), U3.3 (Vin); no longer J3.1
- net at R18.2, U7.1 (PS/SYNC): no longer U7.14 (EN)
- new net: F1.2, J3.1
- new net: F1.1, Q3.1 (D)
- new net +3V3: C8.1, U3.2 (Vout)
- new net 5V_Enable: R10.1, U7.14 (EN)
- no-connect marks 4 -> 0
Other:
- note removed: "Connecting Global \nground by the \nATtiny or manual \nswitch"
- note removed: "Input Power"
- note removed: "Input voltage detection\nfor battery monitoring."
- note removed: "Output\nPower"
- note removed: "RTC"
- note removed: "These devices are always on. All other devices ground are not always conneted. \nThis is so we can power down the raspberry pi and any other peripherals so save power."
- moved on the sheet: C11, C13, C14, C15, C16, C17, C18, C19, C20, J3, L2, R17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

Commit message: Version 4
Parts:
- C11: value 820uF -> 270uF; footprint Capacitors_THT:CP_Radial_D10.0mm_P5.00mm -> Capacitors_THT:CP_Radial_D8.0mm_P3.50mm
Connections:
- net VCC: now also F1.1; no longer C11.1, Q3.3 (S)
- net at J3.1: now also Q3.1 (D); no longer F1.2
- new net: C11.1, F1.2, Q3.3 (S)
Other:
- moved on the sheet: C11, F1, J3, Q3
Changed lines of the file:
@@
 EESchema Schematic File Version 4
 LIBS:pi-hat-cache
-EELAYER 26 0
+EELAYER 29 0
 EELAYER END
 $Descr A4 11693 8268
@@
 L pi-hat-rescue:Connector_Specialized_Jack-DC-pi-hat-cache-pi-hat-rescue J?
 U 1 1 5BCDC42E
-P 850 2150
+P 750 2150
 AR Path="/5BCDC42E" Ref="J?"  Part="1"
 AR Path="/5BCDBE20/5BCDC42E" Ref="J3"  Part="1"
-F 0 "J3" H 928 2475 50  0000 C CNN
-F 1 "Jack-DC" H 928 2384 50  0000 C CNN
-F 2 "Connectors:BARREL_JACK" H 900 2110 50  0001 C CNN
-F 3 "~" H 900 2110 50  0001 C CNN
-F 4 "CP-002A-ND" H 850 2150 50  0001 C CNN "Digikey"
-F 5 "https://www.digikey.com/product-detail/en/cui-inc/PJ-002A/CP-002A-ND/96962" H -200 -400 50  0001 C CNN "Link"
-F 6 "PJ-002A" H -200 -400 50  0001 C CNN "MPN"
-F 7 "DC-005" H -200 -400 50  0001 C CNN "OPL"
-	1    850  2150
+F 0 "J3" H 828 2475 50  0000 C CNN
+F 1 "Jack-DC" H 828 2384 50  0000 C CNN
+F 2 "Connectors:BARREL_JACK" H 800 2110 50  0001 C CNN
+F 3 "~" H 800 2110 50  0001 C CNN
+F 4 "CP-002A-ND" H 750 2150 50  0001 C CNN "Digikey"
+F 5 "https://www.digikey.com/product-detail/en/cui-inc/PJ-002A/CP-002A-ND/96962" H -300 -400 50  0001 C CNN "Link"
+F 6 "PJ-002A" H -300 -400 50  0001 C CNN "MPN"
+F 7 "DC-005" H -300 -400 50  0001 C CNN "OPL"
+	1    750  2150
 	1    0    0    -1
 $EndComp
@@
 L pi-hat-rescue:CP-Device-pi-hat-rescue C?
 U 1 1 5BCDC46F
-P 2600 2050
+P 2200 2050
 AR Path="/5BCDC46F" Ref="C?"  Part="1"
 AR Path="/5BCDBE20/5BCDC46F" Ref="C11"  Part="1"
-F 0 "C11" H 2718 2096 50  0000 L CNN
-F 1 "820uF" H 2718 2005 50  0000 L CNN
-F 2 "Capacitors_THT:CP_Radial_D10.0mm_P5.00mm" H 2638 1900 50  0001 C CNN
-F 3 "~" H 2600 2050 50  0001 C CNN
-F 4 "1189-2915-ND" H 2600 2050 50  0001 C CNN "Digikey"
-F 5 "https://www.digikey.com/product-detail/en/rubycon/25ZLH820MEFC10X20/1189-2915-ND/3563817" H 850 -400 50  0001 C CNN "Link"
-F 6 "25ZLH820MEFC10X20" H 850 -400 50  0001 C CNN "MPN"
-	1    2600 2050
+F 0 "C11" H 2318 2096 50  0000 L CNN
+F 1 "270uF" H 2318 2005 50  0000 L CNN
+F 2 "Capacitors_THT:CP_Radial_D8.0mm_P3.50mm" H 2238 1900 50  0001 C CNN
+F 3 "~" H 2200 2050 50  0001 C CNN
+F 4 "1189-2915-ND" H 2200 2050 50  0001 C CNN "Digikey"
+F 5 "https://www.digikey.com/product-detail/en/rubycon/25ZLH820MEFC10X20/1189-2915-ND/3563817" H 450 -400 50  0001 C CNN "Link"
+F 6 "25ZLH820MEFC10X20" H 450 -400 50  0001 C CNN "MPN"
+	1    2200 2050
 	1    0    0    -1
 $EndComp
@@
 L power:VCC #PWR?
 U 1 1 5BCDC47F
-P 2600 1850
+P 2900 1850
 AR Path="/5BCDC47F" Ref="#PWR?"  Part="1"
 AR Path="/5BCDBE20/5BCDC47F" Ref="#PWR020"  Part="1"
-F 0 "#PWR020" H 2600 1700 50  0001 C CNN
-F 1 "VCC" H 2617 2023 50  0000 C CNN
-F 2 "" H 2600 1850 50  0001 C CNN
-F 3 "" H 2600 1850 50  0001 C CNN
-	1    2600 1850
-	1    0    0    -1
-$EndComp
-Wire Wire Line
-	1150 2050 1200 2050
-Wire Wire Line
-	1150 2150 1200 2150
-Wire Wire Line
-	1200 2150 1200 2250
-Wire Wire Line
-	1150 2250 1200 2250
-Connection ~ 1200 2250
+F 0 "#PWR020" H 2900 1700 50  0001 C CNN
+F 1 "VCC" H 2917 2023 50  0000 C CNN
+F 2 "" H 2900 1850 50  0001 C CNN
+F 3 "" H 2900 1850 50  0001 C CNN
+	1    2900 1850
+	1    0    0    -1
+$EndComp
+Wire Wire Line
+	1050 2050 1100 2050
+Wire Wire Line
+	1050 2150 1100 2150
+Wire Wire Line
+	1100 2150 1100 2250
+Wire Wire Line
+	1050 2250 1100 2250
+Connection ~ 1100 2250
 $Comp
 L power:VCC #PWR?
@@
 L Device:Q_PMOS_DGS Q3
 U 1 1 5C89C5A4
-P 1950 2000
-F 0 "Q3" V 2293 2000 50  0000 C CNN
-F 1 "Q_PMOS_DGS" V 2202 2000 50  0000 C CNN
-F 2 "digikey-footprints:IRF9310PbF" H 2150 2100 50  0001 C CNN
-F 3 "~" H 1950 2000 50  0001 C CNN
-F 4 "IRF9310TRPBFCT-ND" H 0   0   50  0001 C CNN "Digikey"
-F 5 "https://www.digikey.com/products/en?keywords=IRF9310TRPBFCT-ND" H 0   0   50  0001 C CNN "Link"
-F 6 "IRF9310TRPBF" H 0   0   50  0001 C CNN "MPN"
-	1    1950 2000
+P 1550 2000
+F 0 "Q3" V 1893 2000 50  0000 C CNN
+F 1 "Q_PMOS_DGS" V 1802 2000 50  0000 C CNN
+F 2 "digikey-footprints:IRF9310PbF" H 1750 2100 50  0001 C CNN
+F 3 "~" H 1550 2000 50  0001 C CNN
+F 4 "IRF9310TRPBFCT-ND" H -400 0   50  0001 C CNN "Digikey"
+F 5 "https://www.digikey.com/products/en?keywords=IRF9310TRPBFCT-ND" H -400 0   50  0001 C CNN "Link"
+F 6 "IRF9310TRPBF" H -400 0   50  0001 C CNN "MPN"
+	1    1550 2000
 	0    -1   -1   0
 $EndComp
@@
 L Device:Fuse F1
 U 1 1 5C8B932A
-P 1450 1900
-F 0 "F1" V 1253 1900 50  0000 C CNN
-F 1 "Fuse" V 1344 1900 50  0000 C CNN
-F 2 "Resistors_SMD:R_0603_HandSoldering" V 1380 1900 50  0001 C CNN
-F 3 "~" H 1450 1900 50  0001 C CNN
-F 4 "P15125CT-ND" H 0   0   50  0001 C CNN "Digikey"
-F 5 "https://www.digikey.com/product-detail/en/panasonic-electronic-components/ERB-RE5R00V/P15125CT-ND/2796832" H 0   0   50  0001 C CNN "Link"
-F 6 "ERB-RE5R00V" H 0   0   50  0001 C CNN "MPN"
-	1    1450 1900
+P 2550 1900
+F 0 "F1" V 2353 1900 50  0000 C CNN
+F 1 "Fuse" V 2444 1900 50  0000 C CNN
+F 2 "Resistors_SMD:R_0603_HandSoldering" V 2480 1900 50  0001 C CNN
+F 3 "~" H 2550 1900 50  0001 C CNN
+F 4 "P15125CT-ND" H 1100 0   50  0001 C CNN "Digikey"
+F 5 "https://www.digikey.com/product-detail/en/panasonic-electronic-components/ERB-RE5R00V/P15125CT-ND/2796832" H 1100 0   50  0001 C CNN "Link"
+F 6 "ERB-RE5R00V" H 1100 0   50  0001 C CNN "MPN"
+	1    2550 1900
 	0    1    1    0
 $EndComp
@@
 	7350 2250 8250 2250
 Wire Wire Line
-	1200 2250 1950 2250
-Wire Wire Line
-	1200 2050 1200 1900
-Wire Wire Line
-	1200 1900 1300 1900
-Wire Wire Line
-	1600 1900 1750 1900
-Wire Wire Line
-	2150 1900 2600 1900
-Wire Wire Line
-	1950 2200 1950 2250
-Connection ~ 1950 2250
-Wire Wire Line
-	1950 2250 2250 2250
-Wire Wire Line
-	2600 2250 2600 2200
-Wire Wire Line
-	2600 1900 2600 1850
-Connection ~ 2600 1900
-Wire Wire Line
 	4300 2300 4300 2250
 Connection ~ 4300 2250
@@
 L power:GND #PWR019
 U 1 1 5C9FE107
-P 2250 2300
-F 0 "#PWR019" H 2250 2050 50  0001 C CNN
-F 1 "GND" H 2255 2127 50  0000 C CNN
-F 2 "" H 2250 2300 50  0001 C CNN
-F 3 "" H 2250 2300 50  0001 C CNN
-	1    2250 2300
-	1    0    0    -1
-$EndComp
-Wire Wire Line
-	2250 2300 2250 2250
-Connection ~ 2250 2250
-Wire Wire Line
-	2250 2250 2600 2250
+P 2800 2300
+F 0 "#PWR019" H 2800 2050 50  0001 C CNN
+F 1 "GND" H 2805 2127 50  0000 C CNN
+F 2 "" H 2800 2300 50  0001 C CNN
+F 3 "" H 2800 2300 50  0001 C CNN
+	1    2800 2300
+	1    0    0    -1
+$EndComp
+Wire Wire Line
+	2800 2300 2800 2250
 Text HLabel 7950 1000 2    50   Input ~ 0
 5V_Enable
@@
 L power:PWR_FLAG #FLG0102
 U 1 1 5CF57122
-P 1200 1850
-F 0 "#FLG0102" H 1200 1925 50  0001 C CNN
-F 1 "PWR_FLAG" H 1200 2024 50  0000 C CNN
-F 2 "" H 1200 1850 50  0001 C CNN
-F 3 "" H 1200 1850 50  0001 C CNN
-	1    1200 1850
-	1    0    0    -1
-$EndComp
-Wire Wire Line
-	1200 1900 1200 1850
-Connection ~ 1200 1900
+P 1100 1850
+F 0 "#FLG0102" H 1100 1925 50  0001 C CNN
+F 1 "PWR_FLAG" H 1100 2024 50  0000 C CNN
+F 2 "" H 1100 1850 50  0001 C CNN
+F 3 "" H 1100 1850 50  0001 C CNN
+	1    1100 1850
+	1    0    0    -1
+$EndComp
 $Comp
 L Device:R R10
@@
 	8250 1450 8250 1800
 Connection ~ 8250 1800
+Wire Wire Line
+	1100 2250 1550 2250
+Wire Wire Line
+	1550 2200 1550 2250
+Connection ~ 1550 2250
+Wire Wire Line
+	2700 1900 2900 1900
+Wire Wire Line
+	2900 1900 2900 1850
+Connection ~ 2200 1900
+Wire Wire Line
+	1550 2250 2200 2250
+Wire Wire Line
+	2200 2200 2200 2250
+Connection ~ 2200 2250
+Wire Wire Line
+	2200 2250 2800 2250
+Wire Wire Line
+	1100 1850 1100 1900
+Wire Wire Line
+	2200 1900 2400 1900
+Wire Wire Line
+	1750 1900 2200 1900
+Wire Wire Line
+	1350 1900 1100 1900
+Connection ~ 1100 1900
+Wire Wire Line
+	1100 1900 1100 2050
 $EndSCHEMATC
