File: pi-hat.sch (KiCad schematic (older format))
At the start: 41 parts, among them J1 Raspberry_Pi_2_3, J2 Conn_SPI, J3 Conn_RTC, J4 Conn_01x08, J5 USB_B, J7 USB_OUT, J8 Jack-DC, M1 Motor_Servo, M2 Motor_Servo, M3 Motor_Servo, Q1 Q_NMOS_GDS, Q2 Q_NMOS_GDS, Q4 Q_NMOS_GDS, Q5 Q_NMOS_GDS, SW1 SW_Push, SW2 SW_Push, SW3 SW_DPST_x2, U1 ATTINY85-20SU

Commit message: updated pi hat to latest version.
Parts:
- removed C1: CP, Capacitor_THT:CP_Radial_D8.0mm_P3.50mm, symbol Device:CP
- removed D2, D4, D6, D8: LED, LED_SMD:LED_1206_3216Metric_Pad1.07x1.80mm_HandSolder, symbol Device:LED
- removed D3, D7: LED, Connector_JST:JST_XH_B02B-XH-A_1x02_P2.50mm_Vertical, symbol Device:LED
- removed J3: Conn_RTC, Connector_PinHeader_2.54mm:PinHeader_1x04_P2.54mm_Vertical, symbol Connector_Generic:Conn_01x04
- removed J8: Jack-DC, Connector_BarrelJack:BarrelJack_Horizontal, symbol Connector_Specialized:Jack-DC
- removed M1, M2, M3: Motor_Servo, Connector_PinHeader_2.54mm:PinHeader_1x03_P2.54mm_Vertical, symbol Motor:Motor_Servo
- removed MK1, MK2: Mounting_Hole, MountingHole:MountingHole_2.7mm_M2.5, symbol Mechanical:Mounting_Hole
- removed Q2: Q_NMOS_GDS, Package_TO_SOT_SMD:SC-59, symbol Device:Q_NMOS_GSD
- removed Q4: Q_NMOS_GDS, Package_TO_SOT_SMD:SOT-223, symbol Device:Q_NMOS_GDS
- removed R1, R10, R14, R2: 100K, Resistor_SMD:R_1206_3216Metric_Pad1.24x1.80mm_HandSolder, symbol Device:R
- removed R11: 100R, Resistor_SMD:R_1206_3216Metric_Pad1.24x1.80mm_HandSolder, symbol Device:R
- removed R13, R4, R5, R6, R9: 470R, Resistor_SMD:R_1206_3216Metric_Pad1.24x1.80mm_HandSolder, symbol Device:R
- removed SW1, SW2: SW_Push, Connector_JST:JST_XH_B02B-XH-A_1x02_P2.50mm_Vertical, symbol Switch:SW_Push
- removed SW3: SW_DPST_x2, switch-footprint:CJS-1200A1, symbol Switch:SW_DPST_x2
- removed U1: ATTINY85-20SU, Package_DIP:DIP-8_W7.62mm_Socket, symbol MCU_Atmel_ATTINY:ATTINY85-20SU
- added C3, C5: 10uF, Capacitors_SMD:C_0805_HandSoldering, symbol device:C_Small
- added C4: 100nF, Capacitors_SMD:C_0805_HandSoldering, symbol device:C_Small
- added J6: Conn_01x02, Connectors:bornier2, symbol conn:Conn_01x02
- added J9: Conn_01x02, Connectors_JST:JST_XH_B02B-XH-A_02x2.50mm_Straight, symbol conn:Conn_01x02
- added R12: 634K, Resistors_SMD:R_0603_HandSoldering, symbol device:R
- added R2: 470R, Resistors_SMD:R_0603_HandSoldering, symbol pi-hat-rescue:R-Device
- added R7: 100K, Resistors_SMD:R_0603_HandSoldering, symbol device:R
- added U2: MAX98357, Housings_DFN_QFN:QFN-16-1EP_3x3mm_Pitch0.5mm, symbol cacophony-pi-hat:MAX98357
- D1: footprint Connector_JST:JST_XH_B02B-XH-A_1x02_P2.50mm_Vertical -> LEDs:LED_0603_HandSoldering; symbol Device:LED -> pi-hat-rescue:LED-Device; Digikey (none) -> 160-1447-1-ND
- J1: footprint Connector_PinHeader_2.54mm:PinHeader_2x20_P2.54mm_Vertical -> Pin_Headers:Pin_Header_Straight_2x20_Pitch2.54mm; symbol Connector_Specialized:Raspberry_Pi_2_3 -> pi-hat-rescue:Connector_Specialized_Raspberry_Pi_2_3-pi-hat-cache
- J2: footprint Connector_JST:JST_XH_B04B-XH-A_1x04_P2.50mm_Vertical -> Connectors_JST:JST_XH_B04B-XH-A_04x2.50mm_Straight; symbol Connector_Generic:Conn_01x04 -> pi-hat-rescue:Conn_01x04-Connector_Generic
- J4: footprint Connector_JST:JST_XH_B08B-XH-A_1x08_P2.50mm_Vertical -> Connectors_JST:JST_XH_B08B-XH-A_08x2.50mm_Straight; symbol Connector_Generic:Conn_01x08 -> pi-hat-rescue:Conn_01x08-Connector_Generic
- J5: symbol Connector_Specialized:USB_B -> pi-hat-rescue:Connector_Specialized_USB_B-pi-hat-cache
- J7: symbol Connector_Specialized:USB_A -> pi-hat-rescue:Connector_Specialized_USB_A-pi-hat-cache
- Q1, Q5: footprint Package_TO_SOT_SMD:SC-59 -> TO_SOT_Packages_SMD:SC-59_Handsoldering; symbol Device:Q_NMOS_GSD -> pi-hat-rescue:Q_NMOS_GSD-Device
- R15, R3, R8: footprint Resistor_SMD:R_1206_3216Metric_Pad1.24x1.80mm_HandSolder -> Resistors_SMD:R_0603_HandSoldering; symbol Device:R -> pi-hat-rescue:R-Device
Connections:
- net labels added: I2S_BCLK, I2S_DIN, I2S_LRCLK, SPI_CEO, SPI_MISO, SPI_MOSI, SPI_SCLK, THERMAL_POWER, USB_POWER
- net labels removed: Button1, Button2, CameraPower, LED2, Laser, ServoPan, ServoTilt, ServoTrigger, USBPower
- wire segments 163 -> 125
- no-connect marks 18 -> 22
Other:
- note added: "Audio Out"
- note added: "General purpose \nI2C connector"
- note added: "Indication LEDs"
- note added: "Raspberry Pi"
- note added: "Thermal Camera"
- note added: "USB power controll \nfor USB modem"
- note removed: "Gound connection is controller by switch or attiny85\n"

Commit message: Added link, MPN, and Digikey number to all parts.
Parts:
- C3, C5: Digikey (none) -> 1276-2891-1-ND; Link (none) -> https://www.digikey.com/product-detail/en/samsung-electro-m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; MPN (none) -> CL21A106KAYNNNE
- C4: Digikey (none) -> 720-1756-1-ND; Link (none) -> https://www.digikey.com/product-detail/en/vishay-vitramon/V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; MPN (none) -> VJ0805Y104MXXAT
- D1: symbol pi-hat-rescue:LED-Device -> pi-hat-rescue:LED-Device-pi-hat-rescue; Link (none) -> https://www.digikey.com/product-detail/en/lite-on-inc/LTST-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; MPN (none) -> LTST-C191KRKT
- J1: symbol pi-hat-rescue:Connector_Specialized_Raspberry_Pi_2_3-pi-hat-cache -> pi-hat-rescue:Connector_Specialized_Raspberry_Pi_2_3-pi-hat-cache-pi-hat-rescue; Digikey (none) -> S6104-ND; Link (none) -> https://www.digikey.com/product-detail/en/sullins-connector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; MPN (none) -> PPTC202LFBN-RC
- J2: symbol pi-hat-rescue:Conn_01x04-Connector_Generic -> pi-hat-rescue:Conn_01x04-Connector_Generic-pi-hat-rescue; Digikey (none) -> 455-2249-ND; Link (none) -> https://www.digikey.com/product-detail/en/jst-sales-america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; MPN (none) -> B4B-XH-A(LF)(SN)
- J4: symbol pi-hat-rescue:Conn_01x08-Connector_Generic -> pi-hat-rescue:Conn_01x08-Connector_Generic-pi-hat-rescue; Digikey (none) -> 455-2251-ND; Link (none) -> https://www.digikey.com/product-detail/en/jst-sales-america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; MPN (none) -> B8B-XH-A(LF)(SN)
- J5: symbol pi-hat-rescue:Connector_Specialized_USB_B-pi-hat-cache -> pi-hat-rescue:Connector_Specialized_USB_B-pi-hat-cache-pi-hat-rescue; Digikey (none) -> ED2983-ND; Link (none) -> https://www.digikey.com/product-detail/en/on-shore-technolo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; MPN (none) -> USB-B1HSB6
- J6: Digikey (none) -> 277-1667-ND; Link (none) -> https://www.digikey.com/product-detail/en/phoenix-contact/1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; MPN (none) -> 1935161
- J7: symbol pi-hat-rescue:Connector_Specialized_USB_A-pi-hat-cache -> pi-hat-rescue:Connector_Specialized_USB_A-pi-hat-cache-pi-hat-rescue; Digikey (none) -> ED2989-ND; Link (none) -> https://www.digikey.com/product-detail/en/on-shore-technolo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; MPN (none) -> USB-A1HSW6
- J9: Digikey (none) -> 455-2247-ND; Link (none) -> https://www.digikey.com/product-detail/en/jst-sales-america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; MPN (none) -> B2B-XH-A(LF)(SN)
- Q1, Q5: symbol pi-hat-rescue:Q_NMOS_GSD-Device -> pi-hat-rescue:Q_NMOS_GSD-Device-pi-hat-rescue; Digikey (none) -> 785-1015-1-ND; Link (none) -> https://www.digikey.com/product-detail/en/alpha-omega-semic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; MPN (none) -> AO3422
- R12: Digikey (none) -> 541-634KHCT-ND; Link (none) -> https://www.digikey.com/product-detail/en/vishay-dale/CRCW0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; MPN (none) -> CRCW0603634KFKEA
- R15, R8: symbol pi-hat-rescue:R-Device -> pi-hat-rescue:R-Device-pi-hat-rescue; Digikey (none) -> RR08P100KDCT-ND; Link (none) -> https://www.digikey.com/product-detail/en/susumu/RR0816P-10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; MPN (none) -> RR0816P-104-D
- R2, R3: symbol pi-hat-rescue:R-Device -> pi-hat-rescue:R-Device-pi-hat-rescue; Digikey (none) -> 311-470HRCT-ND; Link (none) -> https://www.digikey.com/product-detail/en/yageo/RC0603FR-07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; MPN (none) -> RC0603FR-07470RL
- R7: Digikey (none) -> RR08P100KDCT-ND; Link (none) -> https://www.digikey.com/product-detail/en/susumu/RR0816P-10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; MPN (none) -> RR0816P-104-D
- U2: Digikey (none) -> MAX98357AETE+TCT-ND; Link (none) -> https://www.digikey.com/product-detail/en/maxim-integrated/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; MPN (none) -> MAX98357AETE+T
Changed lines of the file:
@@
 $EndDescr
 $Comp
-L pi-hat-rescue:Connector_Specialized_Raspberry_Pi_2_3-pi-hat-cache J1
+L pi-hat-rescue:Connector_Specialized_Raspberry_Pi_2_3-pi-hat-cache-pi-hat-rescue J1
 U 1 1 5A90DE17
 P 2400 6100
@@
 F 2 "Pin_Headers:Pin_Header_Straight_2x20_Pitch2.54mm" H 3400 7350 50  0001 C CNN
 F 3 "https://www.raspberrypi.org/documentation/hardware/raspberrypi/schematics/RPI-3B-V1_2-SCHEMATIC-REDUCED.pdf" H 2450 5950 50  0001 C CNN
+F 4 "S6104-ND" H 0   0   50  0001 C CNN "Digikey"
+F 5 "https://www.digikey.com/product-detail/en/sullins-connector-solutions/PPTC202LFBN-RC/S6104-ND/807240" H 0   0   50  0001 C CNN "Link"
+F 6 "PPTC202LFBN-RC" H 0   0   50  0001 C CNN "MPN"
 	1    2400 6100
 	1    0    0    -1
 $EndComp
 $Comp
-L pi-hat-rescue:Conn_01x04-Connector_Generic J2
+L pi-hat-rescue:Conn_01x04-Connector_Generic-pi-hat-rescue J2
 U 1 1 5A90E091
 P 3300 3550
@@
 F 2 "Connectors_JST:JST_XH_B04B-XH-A_04x2.50mm_Straight" H 3300 3550 50  0001 C CNN
 F 3 "~" H 3300 3550 50  0001 C CNN
+F 4 "455-2249-ND" H 0   0   50  0001 C CNN "Digikey"
+F 5 "https://www.digikey.com/product-detail/en/jst-sales-america-inc/B4B-XH-A(LF)(SN)/455-2249-ND/1651047" H 0   0   50  0001 C CNN "Link"
+F 6 "B4B-XH-A(LF)(SN)" H 0   0   50  0001 C CNN "MPN"
 	1    3300 3550
 	-1   0    0    1
@@
 	2600 7450 2700 7450
 $Comp
-L pi-hat-rescue:Conn_01x08-Connector_Generic J4
+L pi-hat-rescue:Conn_01x08-Connector_Generic-pi-hat-rescue J4
 U 1 1 5A91824A
 P 2450 1350
@@
 F 2 "Connectors_JST:JST_XH_B08B-XH-A_08x2.50mm_Straight" H 2450 1350 50  0001 C CNN
 F 3 "~" H 2450 1350 50  0001 C CNN
+F 4 "455-2251-ND" H 0   0   50  0001 C CNN "Digikey"
+F 5 "https://www.digikey.com/product-detail/en/jst-sales-america-inc/B8B-XH-A(LF)(SN)/455-2251-ND/1651049" H 0   0   50  0001 C CNN "Link"
+F 6 "B8B-XH-A(LF)(SN)" H 0   0   50  0001 C CNN "MPN"
 	1    2450 1350
 	1    0    0    -1
@@
 $EndComp
 $Comp
-L pi-hat-rescue:R-Device R8
+L pi-hat-rescue:R-Device-pi-hat-rescue R8
 U 1 1 5A9301C4
 P 1350 2050
@@
 F 2 "Resistors_SMD:R_0603_HandSoldering" V 1280 2050 50  0001 C CNN
 F 3 "~" H 1350 2050 50  0001 C CNN
+F 4 "RR08P100KDCT-ND" H 0   0   50  0001 C CNN "Digikey"
+F 5 "https://www.digikey.com/product-detail/en/susumu/RR0816P-104-D/RR08P100KDCT-ND/432772" H 0   0   50  0001 C CNN "Link"
+F 6 "RR0816P-104-D" H 0   0   50  0001 C CNN "MPN"
 	1    1350 2050
 	1    0    0    -1
@@
 	3550 3650 3500 3650
 $Comp
-L pi-hat-rescue:Q_NMOS_GSD-Device Q1
+L pi-hat-rescue:Q_NMOS_GSD-Device-pi-hat-rescue Q1
 U 1 1 5A952EAF
 P 1600 1850
@@
 F 2 "TO_SOT_Packages_SMD:SC-59_Handsoldering" H 1800 1950 50  0001 C CNN
 F 3 "~" H 1600 1850 50  0001 C CNN
+F 4 "785-1015-1-ND" H 0   0   50  0001 C CNN "Digikey"
+F 5 "https://www.digikey.com/product-detail/en/alpha-omega-semiconductor-inc/AO3422/785-1015-1-ND/1855957" H 0   0   50  0001 C CNN "Link"
+F 6 "AO3422" H 0   0   50  0001 C CNN "MPN"
 	1    1600 1850
 	1    0    0    -1
@@
 NoConn ~ 1500 6900
 $Comp
-L pi-hat-rescue:Connector_Specialized_USB_A-pi-hat-cache J7
+L pi-hat-rescue:Connector_Specialized_USB_A-pi-hat-cache-pi-hat-rescue J7
 U 1 1 5A9F478E
 P 10300 5000
@@
 F 2 "Connector_USB:USB_A_Horizontal" H 10450 4950 50  0001 C CNN
 F 3 "" H 10450 4950 50  0001 C CNN
+F 4 "ED2989-ND" H 0   0   50  0001 C CNN "Digikey"
+F 5 "https://www.digikey.com/product-detail/en/on-shore-technology-inc/USB-A1HSW6/ED2989-ND/2677750" H 0   0   50  0001 C CNN "Link"
+F 6 "USB-A1HSW6" H 0   0   50  0001 C CNN "MPN"
 	1    10300 5000
 	1    0    0    -1
@@
 $EndComp
 $Comp
-L pi-hat-rescue:R-Device R15
+L pi-hat-rescue:R-Device-pi-hat-rescue R15
 U 1 1 5AA1C4C6
 P 9950 5900
@@
 F 2 "Resistors_SMD:R_0603_HandSoldering" V 9880 5900 50  0001 C CNN
 F 3 "~" H 9950 5900 50  0001 C CNN
+F 4 "RR08P100KDCT-ND" H 0   0   50  0001 C CNN "Digikey"
+F 5 "https://www.digikey.com/product-detail/en/susumu/RR0816P-104-D/RR08P100KDCT-ND/432772" H 0   0   50  0001 C CNN "Link"
+F 6 "RR0816P-104-D" H 0   0   50  0001 C CNN "MPN"
 	1    9950 5900
 	1    0    0    -1
@@
 	10300 6100 10300 5900
 $Comp
-L pi-hat-rescue:Q_NMOS_GSD-Device Q5
+L pi-hat-rescue:Q_NMOS_GSD-Device-pi-hat-rescue Q5
 U 1 1 5AA1C4D7
 P 10200 5700
@@
 F 2 "TO_SOT_Packages_SMD:SC-59_Handsoldering" H 10400 5800 50  0001 C CNN
 F 3 "~" H 10200 5700 50  0001 C CNN
+F 4 "785-1015-1-ND" H 0   0   50  0001 C CNN "Digikey"
+F 5 "https://www.digikey.com/product-detail/en/alpha-omega-semiconductor-inc/AO3422/785-1015-1-ND/1855957" H 0   0   50  0001 C CNN "Link"
+F 6 "AO3422" H 0   0   50  0001 C CNN "MPN"
 	1    10200 5700
 	1    0    0    -1
@@
 $EndComp
 $Comp
-L pi-hat-rescue:R-Device R3
+L pi-hat-rescue:R-Device-pi-hat-rescue R3
 U 1 1 5AA5DD68
 P 9800 1800
@@
 F 2 "Resistors_SMD:R_0603_HandSoldering" V 9730 1800 50  0001 C CNN
 F 3 "~" H 9800 1800 50  0001 C CNN
+F 4 "311-470HRCT-ND" H 0   0   50  0001 C CNN "Digikey"
+F 5 "https://www.digikey.com/product-detail/en/yageo/RC0603FR-07470RL/311-470HRCT-ND/730203" H 0   0   50  0001 C CNN "Link"
+F 6 "RC0603FR-07470RL" H 0   0   50  0001 C CNN "MPN"
 	1    9800 1800
 	1    0    0    -1
 $EndComp
 $Comp
-L pi-hat-rescue:LED-Device D1
+L pi-hat-rescue:LED-Device-pi-hat-rescue D1
 U 1 1 5AA5DD6F
 P 9800 1450
@@
 F 3 "~" H 9800 1450 50  0001 C CNN
 F 4 "160-1447-1-ND" V 9800 1450 50  0001 C CNN "Digikey"
+F 5 "https://www.digikey.com/product-detail/en/lite-on-inc/LTST-C191KRKT/160-1447-1-ND/386836" H 0   0   50  0001 C CNN "Link"
+F 6 "LTST-C191KRKT" H 0   0   50  0001 C CNN "MPN"
 	1    9800 1450
 	0    -1   -1   0
@@
 	9800 1950 9800 2000
 $Comp
-L pi-hat-rescue:Connector_Specialized_USB_B-pi-hat-cache J5
+L pi-hat-rescue:Connector_Specialized_USB_B-pi-hat-cache-pi-hat-rescue J5
 U 1 1 5AAC3C74
 P 10300 3850
@@
 F 2 "Connector_USB:USB_B_Horizontal" H 10450 3800 50  0001 C CNN
 F 3 "" H 10450 3800 50  0001 C CNN
+F 4 "ED2983-ND" H 0   0   50  0001 C CNN "Digikey"
+F 5 "https://www.digikey.com/product-detail/en/on-shore-technology-inc/USB-B1HSB6/ED2983-ND/2677744" H 0   0   50  0001 C CNN "Link"
+F 6 "USB-B1HSB6" H 0   0   50  0001 C CNN "MPN"
 	1    10300 3850
 	1    0    0    -1
@@
 F 2 "Housings_DFN_QFN:QFN-16-1EP_3x3mm_Pitch0.5mm" H 4950 1400 50  0001 C CNN
 F 3 "" H 4950 1400 50  0001 C CNN
+F 4 "MAX98357AETE+TCT-ND" H 0   0   50  0001 C CNN "Digikey"
+F 5 "https://www.digikey.com/product-detail/en/maxim-integrated/MAX98357AETE-T/MAX98357AETE-TCT-ND/7603777" H 0   0   50  0001 C CNN "Link"
+F 6 "MAX98357AETE+T" H 0   0   50  0001 C CNN "MPN"
 	1    4950 1400
 	1    0    0    -1
@@
 F 2 "Resistors_SMD:R_0603_HandSoldering" V 3980 1250 50  0001 C CNN
 F 3 "" H 4050 1250 50  0001 C CNN
+F 4 "RR08P100KDCT-ND" H 0   0   50  0001 C CNN "Digikey"
+F 5 "https://www.digikey.com/product-detail/en/susumu/RR0816P-104-D/RR08P100KDCT-ND/432772" H 0   0   50  0001 C CNN "Link"
+F 6 "RR0816P-104-D" H 0   0   50  0001 C CNN "MPN"
 	1    4050 1250
 	0    1    1    0
@@
 F 2 "Resistors_SMD:R_0603_HandSoldering" V 4030 1450 50  0001 C CNN
 F 3 "" H 4100 1450 50  0001 C CNN
+F 4 "541-634KHCT-ND" H 0   0   50  0001 C CNN "Digikey"
+F 5 "https://www.digikey.com/product-detail/en/vishay-dale/CRCW0603634KFKEA/541-634KHCT-ND/1180130" H 0   0   50  0001 C CNN "Link"
+F 6 "CRCW0603634KFKEA" H 0   0   50  0001 C CNN "MPN"
 	1    4100 1450
 	0    1    1    0
@@
 F 2 "Connectors:bornier2" H 5650 2100 50  0001 C CNN
 F 3 "~" H 5650 2100 50  0001 C CNN
+F 4 "277-1667-ND" H 0   0   50  0001 C CNN "Digikey"
+F 5 "https://www.digikey.com/product-detail/en/phoenix-contact/1935161/277-1667-ND/568614" H 0   0   50  0001 C CNN "Link"
+F 6 "1935161" H 0   0   50  0001 C CNN "MPN"
 	1    5650 2100
 	0    1    1    0
@@
 $EndComp
 $Comp
-L pi-hat-rescue:R-Device R2
+L pi-hat-rescue:R-Device-pi-hat-rescue R2
 U 1 1 5B6A131D
 P 10150 1800
@@
 F 2 "Resistors_SMD:R_0603_HandSoldering" V 10080 1800 50  0001 C CNN
 F 3 "~" H 10150 1800 50  0001 C CNN
+F 4 "311-470HRCT-ND" H 0   0   50  0001 C CNN "Digikey"
+F 5 "https://www.digikey.com/product-detail/en/yageo/RC0603FR-07470RL/311-470HRCT-ND/730203" H 0   0   50  0001 C CNN "Link"
+F 6 "RC0603FR-07470RL" H 0   0   50  0001 C CNN "MPN"
 	1    10150 1800
 	1    0    0    -1
@@
 F 2 "Connectors_JST:JST_XH_B02B-XH-A_02x2.50mm_Straight" H 10350 1400 50  0001 C CNN
 F 3 "~" H 10350 1400 50  0001 C CNN
+F 4 "455-2247-ND" H 0   0   50  0001 C CNN "Digikey"
+F 5 "https://www.digikey.com/product-detail/en/jst-sales-america-inc/B2B-XH-A(LF)(SN)/455-2247-ND/1651045" H 0   0   50  0001 C CNN "Link"
+F 6 "B2B-XH-A(LF)(SN)" H 0   0   50  0001 C CNN "MPN"
 	1    10350 1400
 	1    0    0    -1
@@
 F 2 "Capacitors_SMD:C_0805_HandSoldering" H 4150 2000 50  0001 C CNN
 F 3 "" H 4150 2000 50  0001 C CNN
+F 4 "1276-2891-1-ND" H 0   0   50  0001 C CNN "Digikey"
+F 5 "https://www.digikey.com/product-detail/en/samsung-electro-mechanics/CL21A106KAYNNNE/1276-2891-1-ND/3890977" H 0   0   50  0001 C CNN "Link"
+F 6 "CL21A106KAYNNNE" H 0   0   50  0001 C CNN "MPN"
 	1    4150 2000
 	1    0    0    -1
@@
 F 2 "Capacitors_SMD:C_0805_HandSoldering" H 3800 2000 50  0001 C CNN
 F 3 "" H 3800 2000 50  0001 C CNN
+F 4 "1276-2891-1-ND" H 0   0   50  0001 C CNN "Digikey"
+F 5 "https://www.digikey.com/product-detail/en/samsung-electro-mechanics/CL21A106KAYNNNE/1276-2891-1-ND/3890977" H 0   0   50  0001 C CNN "Link"
+F 6 "CL21A106KAYNNNE" H 0   0   50  0001 C CNN "MPN"
 	1    3800 2000
 	1    0    0    -1
@@
 F 2 "Capacitors_SMD:C_0805_HandSoldering" H 3450 2000 50  0001 C CNN
 F 3 "" H 3450 2000 50  0001 C CNN
+F 4 "720-1756-1-ND" H 0   0   50  0001 C CNN "Digikey"
+F 5 "https://www.digikey.com/product-detail/en/vishay-vitramon/VJ0805Y104MXXAT/720-1756-1-ND/8324176" H 0   0   50  0001 C CNN "Link"
+F 6 "VJ0805Y104MXXAT" H 0   0   50  0001 C CNN "MPN"
 	1    3450 2000
 	1    0    0    -1

Commit message: Added some Seeed OPL parts
Parts:
- C3, C5: OPL (none) -> CC0805KKX5R8BB106
- C4: OPL (none) -> CC0805KRX7R9BB104
- J7: OPL (none) -> ST-USB-003A
- R15, R7, R8: OPL (none) -> RC0603JR-07100KL
- R2, R3: OPL (none) -> RC0603JR-07470RL
Changed lines of the file:
@@
 F 5 "https://www.digikey.com/product-detail/en/susumu/RR0816P-104-D/RR08P100KDCT-ND/432772" H 0   0   50  0001 C CNN "Link"
 F 6 "RR0816P-104-D" H 0   0   50  0001 C CNN "MPN"
+F 7 "RC0603JR-07100KL" H 0   0   50  0001 C CNN "OPL"
 	1    1350 2050
 	1    0    0    -1
@@
 F 5 "https://www.digikey.com/product-detail/en/on-shore-technology-inc/USB-A1HSW6/ED2989-ND/2677750" H 0   0   50  0001 C CNN "Link"
 F 6 "USB-A1HSW6" H 0   0   50  0001 C CNN "MPN"
+F 7 "ST-USB-003A" H 0   0   50  0001 C CNN "OPL"
 	1    10300 5000
 	1    0    0    -1
@@
 F 5 "https://www.digikey.com/product-detail/en/susumu/RR0816P-104-D/RR08P100KDCT-ND/432772" H 0   0   50  0001 C CNN "Link"
 F 6 "RR0816P-104-D" H 0   0   50  0001 C CNN "MPN"
+F 7 "RC0603JR-07100KL" H 0   0   50  0001 C CNN "OPL"
 	1    9950 5900
 	1    0    0    -1
@@
 F 5 "https://www.digikey.com/product-detail/en/yageo/RC0603FR-07470RL/311-470HRCT-ND/730203" H 0   0   50  0001 C CNN "Link"
 F 6 "RC0603FR-07470RL" H 0   0   50  0001 C CNN "MPN"
+F 7 "RC0603JR-07470RL" H 0   0   50  0001 C CNN "OPL"
 	1    9800 1800
 	1    0    0    -1
@@
 F 5 "https://www.digikey.com/product-detail/en/susumu/RR0816P-104-D/RR08P100KDCT-ND/432772" H 0   0   50  0001 C CNN "Link"
 F 6 "RR0816P-104-D" H 0   0   50  0001 C CNN "MPN"
+F 7 "RC0603JR-07100KL" H 0   0   50  0001 C CNN "OPL"
 	1    4050 1250
 	0    1    1    0
@@
 F 5 "https://www.digikey.com/product-detail/en/yageo/RC0603FR-07470RL/311-470HRCT-ND/730203" H 0   0   50  0001 C CNN "Link"
 F 6 "RC0603FR-07470RL" H 0   0   50  0001 C CNN "MPN"
+F 7 "RC0603JR-07470RL" H 0   0   50  0001 C CNN "OPL"
 	1    10150 1800
 	1    0    0    -1
@@
 F 5 "https://www.digikey.com/product-detail/en/samsung-electro-mechanics/CL21A106KAYNNNE/1276-2891-1-ND/3890977" H 0   0   50  0001 C CNN "Link"
 F 6 "CL21A106KAYNNNE" H 0   0   50  0001 C CNN "MPN"
+F 7 "CC0805KKX5R8BB106" H 0   0   50  0001 C CNN "OPL"
 	1    4150 2000
 	1    0    0    -1
@@
 F 5 "https://www.digikey.com/product-detail/en/samsung-electro-mechanics/CL21A106KAYNNNE/1276-2891-1-ND/3890977" H 0   0   50  0001 C CNN "Link"
 F 6 "CL21A106KAYNNNE" H 0   0   50  0001 C CNN "MPN"
+F 7 "CC0805KKX5R8BB106" H 0   0   50  0001 C CNN "OPL"
 	1    3800 2000
 	1    0    0    -1
@@
 F 5 "https://www.digikey.com/product-detail/en/vishay-vitramon/VJ0805Y104MXXAT/720-1756-1-ND/8324176" H 0   0   50  0001 C CNN "Link"
 F 6 "VJ0805Y104MXXAT" H 0   0   50  0001 C CNN "MPN"
+F 7 "CC0805KRX7R9BB104" H 0   0   50  0001 C CNN "OPL"
 	1    3450 2000
 	1    0    0    -1
