File: pi-hat.sch (KiCad schematic (older format))
At the start: 20 parts, among them J1 Raspberry_Pi_2_3, J2 Conn_SPI, J4 Conn_01x08, J5 USB_B, J6 Conn_01x02, J7 USB_OUT, J9 Conn_01x02, Q1 Q_NMOS_GDS, Q5 Q_NMOS_GDS, U2 MAX98357

Commit message: Updated to version 0.3
Parts:
- removed D1: LED, LEDs:LED_0603_HandSoldering, symbol pi-hat-rescue:LED-Device-pi-hat-rescue
- removed J2: Conn_SPI, Connectors_JST:JST_XH_B04B-XH-A_04x2.50mm_Straight, symbol pi-hat-rescue:Conn_01x04-Connector_Generic-pi-hat-rescue
- removed J9: Conn_01x02, Connectors_JST:JST_XH_B02B-XH-A_02x2.50mm_Straight, symbol conn:Conn_01x02
- removed R2, R3: 470R, Resistors_SMD:R_0603_HandSoldering, symbol pi-hat-rescue:R-Device-pi-hat-rescue
- added BT1: 1206, pi-hat-footprints:CR1220, symbol device:Battery_Cell
- added C1, C9: 2.2uF, Capacitors_SMD:C_0603, symbol device:C_Small
- added C2: 10uF, Capacitors_SMD:C_0805, symbol device:C_Small
- added C6: 2.2uF, Capacitors_SMD:C_0603, symbol Device:C
- added D1: D_Zener, Diodes_SMD:D_SOD-323, symbol device:D_Zener
- added D2: LED_RED, LEDs:LED_0603, symbol pi-hat-rescue:LED-Device-pi-hat-rescue
- added J2, J8: Conn_01x04, Connectors_JST:JST_XH_B04B-XH-A_04x2.50mm_Straight, symbol conn:Conn_01x04
- added MK1, MK2: Mounting_Hole, Mounting_Holes:MountingHole_3mm_Pad, symbol Mechanical:Mounting_Hole
- added Q2: Q_NMOS_GSD, TO_SOT_Packages_SMD:SOT-23, symbol pi-hat-rescue:Q_NMOS_GSD-Device-pi-hat-rescue
- added R1, R9: 1K, Resistors_SMD:R_0603, symbol device:R
- added R2: 120R, Resistors_SMD:R_0603, symbol Device:R
- added R3: 100K, Resistors_SMD:R_0603, symbol Device:R
- added R4: 10K, Resistors_SMD:R_0603, symbol device:R
- added R5, R6: 470R, Resistors_SMD:R_0603, symbol pi-hat-rescue:R-Device-pi-hat-rescue
- added U1: MAX485E, Housings_SSOP:MSOP-8_3x3mm_Pitch0.65mm, symbol interface:MAX485E
- added U4: ATTINY85-20SU, Housings_DIP:DIP-8_W7.62mm_Socket, symbol pi-hat-rescue:ATTINY85-20SU-pi-hat-cache-pi-hat-rescue
- added U5: PCF8523, Housings_SOIC:SOIC-8_3.9x4.9mm_Pitch1.27mm, symbol cacophony-pi-hat:PCF8523
- added Y1: 32.768, Crystals:Crystal_SMD_SeikoEpson_MC306-4pin_8.0x3.2mm, symbol device:Crystal_GND23
- C3, C4, C5: footprint Capacitors_SMD:C_0805_HandSoldering -> Capacitors_SMD:C_0805
- J4: OPL (none) -> B8B-XH-A(LF)(SN)
- J6: OPL (none) -> 1725656
- Q1, Q5: value Q_NMOS_GDS -> Q_NMOS_GSD; footprint TO_SOT_Packages_SMD:SC-59_Handsoldering -> TO_SOT_Packages_SMD:SOT-23; Digikey 785-1015-1-ND -> 785-1009-1-ND; Link https://www.digikey.com/product-detail/en/alpha-omega-semiconductor-inc/AO3422/785-1015-1-ND/1855957 -> https://www.digikey.com/product-detail/en/alpha-omega-semiconductor-inc/AO3414/785-1009-1-ND/1855951; MPN AO3422 -> AO3414
- R12: footprint Resistors_SMD:R_0603_HandSoldering -> Resistors_SMD:R_0603
- R15, R7, R8: footprint Resistors_SMD:R_0603_HandSoldering -> Resistors_SMD:R_0603; OPL RC0603JR-07100KL -> (none)
Connections:
- net +5V: now also C6.1, U1.8 (VCC); no longer J4.6 (Pin_6)
- net GND: now also BT1.2 (-), C1.2, C2.2, C6.2, C9.2, D2.1 (K), J8.1 (Pin_1), J8.2 (Pin_2), Q2.2 (S), R3.2, R4.2, U1.5 (GND), U4.4 (GND), U5.4 (VSS)
- net SCL: now also U4.7 (PB2(SCK/USCK/SCL/T0/INT0/ADC1/PCINT2)), U5.6 (SCL)
- net SDA: now also U4.5 (PB0(MOSI/DI/SDA/AIN0/OC0A/~OC1A~/AREF/PCINT0)), U5.5 (SDA)
- net RPi_3V3: now reaches J1.1 (3V3)
- net RPi_3V3: now also J1.17 (3V3), J4.6 (Pin_6)
- net Rx: now reaches J1.10 ((RXD0)_GPIO15)
- net Rx: now also U1.4 (DI)
- net Tx_enable: now reaches J1.11 (GPIO17_(GEN0))
- net Tx_enable: now also U1.2 (~RE), U1.3 (DE)
- net Tx: now reaches J1.8 ((TXD0)_GPIO14)
- net Tx: now also U1.1 (RO)
- net LED1: no longer names the net of J1.38 (GPIO20)
- new net: J2.1 (Pin_1), R2.2, U1.6 (A)
- new net: J2.2 (Pin_2), R2.1, U1.7 (B)
- new net: J2.4 (Pin_4), Q2.3 (D)
- new net: D2.2 (A), R6.2
- new net: D1.2 (A), R1.1
- new net: J8.3 (Pin_3), R5.2
- new net: U5.1 (OSCI), Y1.1
- new net: U5.2 (OSCO), Y1.4
- new net: BT1.1 (+), U5.3 (VBAT)
- new net: C2.1, R9.2, U5.8 (VDD)
- new net +3V3: C9.1, R9.1, U4.8 (VCC)
- new net 5V_Enable: U4.2 (PB3(XTAL1/CLKI/~OC1B~/ADC3/PCINT3))
- new net Battery_Sense: C1.1, R1.2, R4.1, U4.3 (PB4(XTAL2/CLKO/OC1B/ADC2/PCINT4))
- new net Enable_trap: Q2.1 (G), R3.1
- new net LED_Indicator: R5.1, R6.1, U4.6 (PB1(MISO/DO/AIN1/OC0B/OC1A/PCINT1))
- new net Reset: J8.4 (Pin_4), U4.1 (PB5(~RESET~/dW/ADC0/PCINT5))
- new net VCC: D1.1 (K), J2.3 (Pin_3)
- no-connect marks 22 -> 21
Other:
- note added: "RS485"
- note added: "RTC"
- note added: "Reset/LED button"
- note added: "Trap plug"
- note removed: "General purpose \nI2C connector"
- note removed: "Indication LEDs"
- moved on the sheet: J1, J5, J7, Q5, R15

Commit message: Version 4
Parts:
- added FID1, FID2, FID3: FIDUCIAL, Fiducials:Fiducial_1mm_Dia_2.54mm_Outer_CopperTop, symbol mechanical:Mounting_Hole
- BT1: value 1206 -> 1220
- J1: Digikey S6104-ND -> SAM8767-ND; Link https://www.digikey.com/product-detail/en/sullins-connector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 -> https://www.digikey.com/products/en?keywords=SAM8767-ND; MPN PPTC202LFBN-RC -> ESQ-120-14-G-D
- J2: Digikey 455-2249-ND -> 455-1994-ND; Link https://www.digikey.com/product-detail/en/jst-sales-america-inc/B4B-XH-A-LF-SN/455-2249-ND/1651047 -> https://www.digikey.com/product-detail/en/jst-sales-america-inc/B04B-XASK-1-LF-SN/455-1994-ND/1634735; MPN B4B-XH-A(LF)(SN) -> B04B-XASK-1(LF)(SN)
- J4: Digikey 455-2251-ND -> 455-1998-ND; Link https://www.digikey.com/product-detail/en/jst-sales-america-inc/B8B-XH-A(LF)(SN)/455-2251-ND/1651049 -> https://www.digikey.com/product-detail/en/jst-sales-america-inc/B08B-XASK-1-LF-SN/455-1998-ND/1634739; MPN B8B-XH-A(LF)(SN) -> B08B-XASK-1(LF)(SN); OPL B8B-XH-A(LF)(SN) -> (none)
- J6: footprint Connectors:bornier2 -> Connectors_JST:JST_XH_B02B-XH-A_02x2.50mm_Straight; Digikey 277-1667-ND -> 455-1989-ND; Link https://www.digikey.com/product-detail/en/phoenix-contact/1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 -> https://www.digikey.com/product-detail/en/jst-sales-america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; MPN 1935161 -> B02B-XASK-1(LF)(SN); OPL 1725656 -> (none)
- J8: footprint Connectors_JST:JST_XH_B04B-XH-A_04x2.50mm_Straight -> Connectors_JST:JST_PH_B4B-PH-K_04x2.00mm_Straight; Digikey 455-2249-ND -> 455-1706-ND; Link https://www.digikey.com/product-detail/en/jst-sales-america-inc/B4B-XH-A-LF-SN/455-2249-ND/1651047 -> https://www.digikey.com/product-detail/en/jst-sales-america-inc/B4B-PH-K-S-LF-SN/455-1706-ND/926613; MPN B4B-XH-A(LF)(SN) -> B4B-PH-K-S(LF)(SN)
Connections:
- net Enable_trap: now also J1.13 (GPIO27_(GEN2))
- net Rx: now also U1.1 (RO); no longer U1.4 (DI)
- net Tx: now also U1.4 (DI); no longer U1.1 (RO)
- net at U2.10 (OUTN): now also J6.1 (Pin_1); no longer J6.2 (Pin_2)
- net at U2.9 (OUTP): now also J6.2 (Pin_2); no longer J6.1 (Pin_1)
- no-connect marks 21 -> 20
Changed lines of the file:
@@
 EESchema Schematic File Version 4
 LIBS:pi-hat-cache
-EELAYER 26 0
+EELAYER 29 0
 EELAYER END
 $Descr A4 11693 8268
@@
 F 2 "Pin_Headers:Pin_Header_Straight_2x20_Pitch2.54mm" H 3100 7350 50  0001 C CNN
 F 3 "https://www.raspberrypi.org/documentation/hardware/raspberrypi/schematics/RPI-3B-V1_2-SCHEMATIC-REDUCED.pdf" H 2150 5950 50  0001 C CNN
-F 4 "S6104-ND" H -300 0   50  0001 C CNN "Digikey"
-F 5 "https://www.digikey.com/product-detail/en/sullins-connector-solutions/PPTC202LFBN-RC/S6104-ND/807240" H -300 0   50  0001 C CNN "Link"
-F 6 "PPTC202LFBN-RC" H -300 0   50  0001 C CNN "MPN"
+F 4 "SAM8767-ND" H -300 0   50  0001 C CNN "Digikey"
+F 5 "https://www.digikey.com/products/en?keywords=SAM8767-ND" H -300 0   50  0001 C CNN "Link"
+F 6 "ESQ-120-14-G-D" H -300 0   50  0001 C CNN "MPN"
 	1    2100 6100
 	1    0    0    -1
@@
 F 2 "Connectors_JST:JST_XH_B08B-XH-A_08x2.50mm_Straight" H 2450 1350 50  0001 C CNN
 F 3 "~" H 2450 1350 50  0001 C CNN
-F 4 "455-2251-ND" H 0   0   50  0001 C CNN "Digikey"
-F 5 "https://www.digikey.com/product-detail/en/jst-sales-america-inc/B8B-XH-A(LF)(SN)/455-2251-ND/1651049" H 0   0   50  0001 C CNN "Link"
-F 6 "B8B-XH-A(LF)(SN)" H 0   0   50  0001 C CNN "MPN"
-F 7 "B8B-XH-A(LF)(SN)" H 0   0   50  0001 C CNN "OPL"
+F 4 "455-1998-ND" H 0   0   50  0001 C CNN "Digikey"
+F 5 "https://www.digikey.com/product-detail/en/jst-sales-america-inc/B08B-XASK-1-LF-SN/455-1998-ND/1634739" H 0   0   50  0001 C CNN "Link"
+F 6 "B08B-XASK-1(LF)(SN)" H 0   0   50  0001 C CNN "MPN"
 	1    2450 1350
 	1    0    0    -1
@@
 F 0 "J6" H 5730 2092 50  0000 L CNN
 F 1 "Conn_01x02" H 5730 2001 50  0000 L CNN
-F 2 "Connectors:bornier2" H 5650 2100 50  0001 C CNN
+F 2 "Connectors_JST:JST_XH_B02B-XH-A_02x2.50mm_Straight" H 5650 2100 50  0001 C CNN
 F 3 "~" H 5650 2100 50  0001 C CNN
-F 4 "277-1667-ND" H 0   0   50  0001 C CNN "Digikey"
-F 5 "https://www.digikey.com/product-detail/en/phoenix-contact/1935161/277-1667-ND/568614" H 0   0   50  0001 C CNN "Link"
-F 6 "1935161" H 0   0   50  0001 C CNN "MPN"
-F 7 "1725656" H 0   0   50  0001 C CNN "OPL"
+F 4 "455-1989-ND" H 0   0   50  0001 C CNN "Digikey"
+F 5 "https://www.digikey.com/product-detail/en/jst-sales-america-inc/B02B-XASK-1-LF-SN/455-1989-ND/1634730" H 0   0   50  0001 C CNN "Link"
+F 6 "B02B-XASK-1(LF)(SN)" H 0   0   50  0001 C CNN "MPN"
 	1    5650 2100
 	0    1    1    0
@@
 NoConn ~ 1200 6300
 NoConn ~ 1200 6400
-NoConn ~ 1200 6500
-Wire Wire Line
-	5650 1850 5650 1900
-Wire Wire Line
-	5350 1850 5650 1850
-Wire Wire Line
-	5550 1750 5550 1900
-Wire Wire Line
-	5350 1750 5550 1750
 $Comp
 L device:C_Small C3
@@
 Text Label 3950 6350 2    50   ~ 0
 Tx_enable
+Text Label 3950 6500 2    50   ~ 0
+Tx
 Text Label 3950 6200 2    50   ~ 0
-Tx
-Text Label 3950 6500 2    50   ~ 0
 Rx
 $Comp
@@
 F 0 "J8" H 9850 3050 50  0000 R CNN
 F 1 "Conn_01x04" V 9900 3500 50  0000 R CNN
-F 2 "Connectors_JST:JST_XH_B04B-XH-A_04x2.50mm_Straight" H 9800 3350 50  0001 C CNN
+F 2 "Connectors_JST:JST_PH_B4B-PH-K_04x2.00mm_Straight" H 9800 3350 50  0001 C CNN
 F 3 "~" H 9800 3350 50  0001 C CNN
-F 4 "455-2249-ND" H 0   0   50  0001 C CNN "Digikey"
-F 5 "https://www.digikey.com/product-detail/en/jst-sales-america-inc/B4B-XH-A-LF-SN/455-2249-ND/1651047" H 0   0   50  0001 C CNN "Link"
-F 6 "B4B-XH-A(LF)(SN)" H 0   0   50  0001 C CNN "MPN"
+F 4 "455-1706-ND" H 0   0   50  0001 C CNN "Digikey"
+F 5 "https://www.digikey.com/product-detail/en/jst-sales-america-inc/B4B-PH-K-S-LF-SN/455-1706-ND/926613" H 0   0   50  0001 C CNN "Link"
+F 6 "B4B-PH-K-S(LF)(SN)" H 0   0   50  0001 C CNN "MPN"
 	1    9800 3350
 	-1   0    0    1
@@
 AR Path="/5BCDBE20/5CA45D6E" Ref="BT?"  Part="1"
 F 0 "BT1" H 9468 1996 50  0000 L CNN
-F 1 "1206" H 9468 1905 50  0000 L CNN
+F 1 "1220" H 9468 1905 50  0000 L CNN
 F 2 "pi-hat-footprints:CR1220" V 9350 1960 50  0001 C CNN
 F 3 "" V 9350 1960 50  0001 C CNN
@@
 F 2 "Connectors_JST:JST_XH_B04B-XH-A_04x2.50mm_Straight" H 6350 6600 50  0001 C CNN
 F 3 "~" H 6350 6600 50  0001 C CNN
-F 4 "455-2249-ND" H 0   0   50  0001 C CNN "Digikey"
-F 5 "https://www.digikey.com/product-detail/en/jst-sales-america-inc/B4B-XH-A-LF-SN/455-2249-ND/1651047" H 0   0   50  0001 C CNN "Link"
-F 6 "B4B-XH-A(LF)(SN)" H 0   0   50  0001 C CNN "MPN"
+F 4 "455-1994-ND" H 0   0   50  0001 C CNN "Digikey"
+F 5 "https://www.digikey.com/product-detail/en/jst-sales-america-inc/B04B-XASK-1-LF-SN/455-1994-ND/1634735" H 0   0   50  0001 C CNN "Link"
+F 6 "B04B-XASK-1(LF)(SN)" H 0   0   50  0001 C CNN "MPN"
 	1    6350 6600
 	1    0    0    -1
@@
 Wire Wire Line
 	5400 6200 5400 6600
+Text Label 1150 6500 2    50   ~ 0
+Enable_trap
+Wire Wire Line
+	1150 6500 1200 6500
+$Comp
+L mechanical:Mounting_Hole FID1
+U 1 1 5CC30A0D
+P 9600 6300
+F 0 "FID1" H 9700 6346 50  0000 L CNN
+F 1 "FIDUCIAL" H 9700 6255 50  0000 L CNN
+F 2 "Fiducials:Fiducial_1mm_Dia_2.54mm_Outer_CopperTop" H 9600 6300 50  0001 C CNN
+F 3 "" H 9600 6300 50  0001 C CNN
+	1    9600 6300
+	1    0    0    -1
+$EndComp
+$Comp
+L mechanical:Mounting_Hole FID2
+U 1 1 5CC30B76
+P 9600 6050
+F 0 "FID2" H 9700 6096 50  0000 L CNN
+F 1 "FIDUCIAL" H 9700 6005 50  0000 L CNN
+F 2 "Fiducials:Fiducial_1mm_Dia_2.54mm_Outer_CopperTop" H 9600 6050 50  0001 C CNN
+F 3 "" H 9600 6050 50  0001 C CNN
+	1    9600 6050
+	1    0    0    -1
+$EndComp
+$Comp
+L mechanical:Mounting_Hole FID3
+U 1 1 5CC3ABA3
+P 9600 5800
+F 0 "FID3" H 9700 5846 50  0000 L CNN
+F 1 "FIDUCIAL" H 9700 5755 50  0000 L CNN
+F 2 "Fiducials:Fiducial_1mm_Dia_2.54mm_Outer_CopperTop" H 9600 5800 50  0001 C CNN
+F 3 "" H 9600 5800 50  0001 C CNN
+	1    9600 5800
+	1    0    0    -1
+$EndComp
+Wire Wire Line
+	5650 1750 5650 1900
+Wire Wire Line
+	5350 1750 5650 1750
+Wire Wire Line
+	5350 1850 5550 1850
+Wire Wire Line
+	5550 1850 5550 1900
 $EndSCHEMATC
